File: faceboard-7-sensor/facebard-7-sensor-led.brd (EAGLE design)
At the start: 37 x 91.4 mm, 31 parts, among them Q1 QRE1113, Q2 QRE1113, Q3 QRE1113, Q4 QRE1113, Q5 QRE1113, Q6 QRE1113, Q7 QRE1113, U1 CD4051BE

Commit message: add ffc boards
Connections:
- net N$10 renamed C4
- net N$12 renamed C5
- net N$14 renamed C6
- net N$2 renamed C0
- net N$4 renamed C1
- net N$6 renamed C2
- net N$8 renamed C3
Changed lines of the file:
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@@
 <wire x1="2.4184375" y1="1.71" x2="5.1362375" y2="4.4278" width="0.1524" layer="16"/>
 </signal>
-<signal name="N$2">
+<signal name="C0">
 <contactref element="U1" pad="13"/>
 <contactref element="Q1" pad="3"/>
@@
 <wire x1="2.6194" y1="14.8156" x2="5.8937625" y2="14.8156" width="0.1524" layer="1"/>
 </signal>
-<signal name="N$4">
+<signal name="C1">
 <contactref element="Q2" pad="3"/>
 <contactref element="R4" pad="1"/>
@@
 <wire x1="3.735" y1="27.72" x2="7.5" y2="27.72" width="0.1524" layer="1"/>
 </signal>
-<signal name="N$6">
+<signal name="C2">
 <contactref element="Q3" pad="3"/>
 <contactref element="R6" pad="1"/>
@@
 <wire x1="4.855" y1="40.62" x2="7.5" y2="40.62" width="0.1524" layer="1"/>
 </signal>
-<signal name="N$8">
+<signal name="C3">
 <contactref element="Q4" pad="3"/>
 <contactref element="R8" pad="1"/>
@@
 <wire x1="5.975" y1="53.52" x2="7.5" y2="53.52" width="0.1524" layer="1"/>
 </signal>
-<signal name="N$10">
+<signal name="C4">
 <contactref element="Q5" pad="3"/>
 <contactref element="R10" pad="1"/>
@@
 <wire x1="2.11" y1="71.81" x2="7.5" y2="66.42" width="0.1524" layer="1"/>
 </signal>
-<signal name="N$12">
+<signal name="C5">
 <contactref element="Q6" pad="3"/>
 <contactref element="R12" pad="1"/>
@@
 <wire x1="7.5" y1="80.035" x2="7.5" y2="79.32" width="0.1524" layer="1"/>
 </signal>
-<signal name="N$14">
+<signal name="C6">
 <contactref element="Q7" pad="3"/>
 <contactref element="R14" pad="1"/>
