File: faceboard-7-sensor/controller-board-ffc.sch (EAGLE design)
At the start: 42 parts, among them J1 1-1734592-4, J3 1-1734592-4, Q1 QRE1113, Q2 QRE1113, Q3 QRE1113, Q4 QRE1113, Q5 QRE1113, Q6 QRE1113, Q7 QRE1113, U1 CD4051BE

Commit message: add ffc
Parts:
- removed D1, D2, D3, D4, D5, D6, D7: 1655, 1655:1655
- removed FFCIN, FFCOUT: 52806-1410, 52806-1410:52806-1410
- removed J1, J3: 1-1734592-4, 1-1734592-4:1-1734592-4
- removed Q1, Q2, Q3, Q4, Q5, Q6, Q7: QRE1113, qre1113:QRE1113
- removed R1, R11, R13, R3, R5, R7, R9: 100, rcl:R-EU_0207/10
- removed R10, R12, R14, R2, R4, R6, R8: 100k, rcl:R-EU_0207/10
- removed SJ1, SJ2, SJ3, SJ4, SJ5, SJ6, SJ7: (no value), jumper:SJ
- removed SV1: (no value), con-lstb:MA07-1
- removed U1: CD4051BE, CD4051BE:CD4051BE
- added ANALOG: SIGNALS, con-lstb:MA08-1
- added FRAM: FRAM, con-lstb:MA08-1
- added H1: MOUNT-PAD-ROUND2.8, holes:MOUNT-PAD-ROUND2.8
- added H2: MOUNT-PAD-SQUARE2.8, holes:MOUNT-PAD-SQUARE2.8
- added JUMP1, JUMP2: HEADER, con-lstb:MA08-1
- added LEDR: 300, rcl:R-EU_0207/10
- added POWER: POWER, con-lstb:MA04-1
- added RIBBON: 686114148922, 686114148922:686114148922
- added ROTARY: B5B-PH-K, con-jst-ph:B5B-PH-K
- added SERIAL: ARDUINO4, con-lstb:MA07-1
- added U$1: NANO, Arduino-clone:NANO
- SV4: value (none) -> J3; device con-lstb:MA07-1 -> con-lstb:MA03-1
Connections:
- removed net LEDDIN: D1.DIN, FFCIN.7, J1.7
- removed net LEDDOUT: D7.DOUT, FFCOUT.8, J3.8
- removed net N$1: Q1.1, R1.2
- removed net N$11: Q6.1, R11.2
- removed net N$13: Q7.1, R13.2
- removed net N$15: D6.DOUT, D7.DIN
- removed net N$16: D1.DOUT, D2.DIN
- removed net N$17: D2.DOUT, D3.DIN
- removed net N$18: D4.DIN
- removed net N$19: D4.DOUT, D5.DIN
- removed net N$20: D5.DOUT, D6.DIN
- removed net N$5: Q3.1, R5.2
- removed net N$7: Q4.1, R7.2
- removed net N$9: Q5.1, R9.2
- removed net Q1SIG: Q1.3, R2.1, U1.CHANNELSIN/OUT0
- removed net Q2SIG: Q2.3, R4.1, U1.CHANNELSIN/OUT1
- removed net Q3SIG: Q3.3, R6.1, U1.CHANNELSIN/OUT2
- removed net Q4SIG: Q4.3, R8.1, U1.CHANNELSIN/OUT3
- removed net Q5SIG: Q5.3, R10.1, U1.CHANNELSIN/OUT4
- removed net Q6SIG: Q6.3, R12.1, U1.CHANNELSIN/OUT5
- removed net Q7SIG: Q7.3, R14.1, U1.CHANNELSIN/OUT6
- removed net SIG: SJ1.2, SJ2.2, SJ3.2, SJ4.2, SJ5.2, SJ6.2, SJ7.2, SV1.1, SV1.2, SV1.3, SV1.4, SV1.5, SV1.6, SV1.7, U1.COMOUT/IN
- removed net SIG1: FFCIN.8, FFCOUT.7, J1.14, J3.1, SJ1.1, SV4.1
- removed net SIG2: FFCIN.9, FFCOUT.6, J1.13, J3.2, SJ2.1, SV4.2
- removed net SIG3: FFCIN.10, FFCOUT.5, J1.12, J3.3, SJ3.1, SV4.3
- removed net SIG4: FFCIN.11, FFCOUT.4, J1.11, J3.4, SJ4.1, SV4.4
- removed net SIG5: FFCIN.12, FFCOUT.3, J1.10, J3.5, SJ5.1, SV4.5
- removed net SIG6: FFCIN.13, FFCOUT.2, J1.9, J3.6, SJ6.1, SV4.6
- removed net SIG7: FFCIN.14, FFCOUT.1, J1.8, J3.7, SJ7.1, SV4.7
- new net 3.3V: SV4.2, U$1.3.3V
- new net A0: ANALOG.8, RIBBON.1, U$1.A0
- new net A1: ANALOG.7, RIBBON.2, U$1.A1
- new net A2: ANALOG.6, RIBBON.3, U$1.A2
- new net A3: ANALOG.5, RIBBON.4, U$1.A3
- new net A4: ANALOG.4, RIBBON.5, U$1.A4
- new net A5: ANALOG.3, RIBBON.6, U$1.A5
- new net A6: ANALOG.2, RIBBON.7, U$1.A6
- new net A7: ANALOG.1, U$1.A7
- new net AREF: SV4.1, U$1.AREF
- new net D0: SERIAL.7, U$1.TX0
- new net D1: SERIAL.6, U$1.RX1
- new net D13: SV4.3, U$1.D13
- new net D9: LEDR.1, U$1.D9
- new net FRAM_CLK: FRAM.5, U$1.D5
- new net FRAM_CS: FRAM.2, SERIAL.3, U$1.D2
- new net FRAM_MISO: FRAM.4, U$1.D4
- new net FRAM_MOSI: FRAM.3, SERIAL.2, U$1.D3
- new net LEDDATA: LEDR.2, RIBBON.8
- new net N$8: FRAM.1
- new net ROTA: ROTARY.3, U$1.D10
- new net ROTB: ROTARY.2, U$1.D11
- new net ROTC: ROTARY.1, U$1.D12
- new net RST: POWER.3, SERIAL.5, U$1.RST, U$1.RST1
- new net VIN: H1.MOUNT, POWER.1, U$1.RAW
- new net VUSB: POWER.4, U$1.5.5V
- net 3V: now also FRAM.8, RIBBON.13, ROTARY.5; no longer D1.VDD, D2.VDD, D3.VDD, D4.VDD, D5.VDD, D6.VDD, D7.VDD, FFCIN.2, FFCOUT.13, J1.2, J3.13
- net 5V: now also RIBBON.12; no longer FFCIN.3, FFCOUT.12, J1.3, J3.12, R1.1, R10.2, R11.1, R12.2, R13.1, R14.2, R2.2, R3.1, R4.2, R5.1, R6.2, R7.1, R8.2, R9.1, U1.VDD
- net A: now also RIBBON.11, U$1.D6; no longer FFCIN.4, FFCOUT.11, J1.4, J3.11, U1.A
- net B: now also RIBBON.10, U$1.D7; no longer FFCIN.5, FFCOUT.10, J1.5, J3.10, U1.B
- net C: now also RIBBON.9, U$1.D8; no longer FFCIN.6, FFCOUT.9, J1.6, J3.9, U1.C
- net GND: now also FRAM.7, H2.MOUNT, POWER.2, RIBBON.14, RIBBON.MP1, RIBBON.MP2, ROTARY.4, SERIAL.4, U$1.GND, U$1.GND2; no longer D1.VSS, D2.VSS, D3.VSS, D4.VSS, D5.VSS, D6.VSS, D7.VSS, FFCIN.1, FFCOUT.14, J1.1, J3.14, Q1.2, Q1.4, Q2.2, Q2.4, Q3.2, Q3.4, Q4.2, Q4.4, Q5.2, Q5.4, Q6.2, Q6.4, Q7.2, Q7.4, U1.INH, U1.VEE, U1.VSS
- net N$3: now also FRAM.6; no longer Q2.1, R3.2

Commit message: add ffc boards
Parts:
- removed ANALOG: SIGNALS, con-lstb:MA08-1
- removed H1: MOUNT-PAD-ROUND2.8, holes:MOUNT-PAD-ROUND2.8
- removed H2: MOUNT-PAD-SQUARE2.8, holes:MOUNT-PAD-SQUARE2.8
- removed JUMP1, JUMP2: HEADER, con-lstb:MA08-1
- removed POWER: POWER, con-lstb:MA04-1
- removed RIBBON: 686114148922, 686114148922:686114148922
- removed SERIAL: ARDUINO4, con-lstb:MA07-1
- removed SV4: J3, con-lstb:MA03-1
- added FACEBOARD: 52806-1410, 52806-1410:52806-1410
- added J1: DCJ0202, con-jack:DCJ0202
- added RESET: B2B-PH-K, con-jst-ph:B2B-PH-K
- added RIBBON1: 686114148922, 686114148922:686114148922
- FRAM: value FRAM -> MB85RS2MTA
Connections:
- removed net 3.3V: SV4.2, U$1.3.3V
- removed net N$3: FRAM.6
- new net NC3V: FRAM.7
- new net RST0: U$1.RST
- net 3V: now also FACEBOARD.2, RIBBON1.2, U$1.3.3V; no longer RIBBON.13
- net 5V: now also FACEBOARD.3, RIBBON1.3; no longer RIBBON.12
- net A: now also FACEBOARD.4, RIBBON1.4; no longer RIBBON.11
- net A0: now also FACEBOARD.8, RIBBON1.8; no longer ANALOG.8, RIBBON.1
- net A1: now also FACEBOARD.9, RIBBON1.9; no longer ANALOG.7, RIBBON.2
- net A2: now also FACEBOARD.10, RIBBON1.10; no longer ANALOG.6, RIBBON.3
- net A3: now also FACEBOARD.11, RIBBON1.11; no longer ANALOG.5, RIBBON.4
- net A4: now also FACEBOARD.12, RIBBON1.12; no longer ANALOG.4, RIBBON.5
- net A5: now also FACEBOARD.13, RIBBON1.13; no longer ANALOG.3, RIBBON.6
- net A6: now also FACEBOARD.14, RIBBON1.14; no longer ANALOG.2, RIBBON.7
- net A7: no longer ANALOG.1
- net AREF: no longer SV4.1
- net B: now also FACEBOARD.5, RIBBON1.5; no longer RIBBON.10
- net C: now also FACEBOARD.6, RIBBON1.6; no longer RIBBON.9
- net D0: no longer SERIAL.7
- net D1: no longer SERIAL.6
- net D13: no longer SV4.3
- net FRAM_CS: no longer SERIAL.3
- net FRAM_MOSI: no longer SERIAL.2
- net GND: now also FACEBOARD.1, FRAM.6, J1.2, J1.3, RESET.2, RIBBON1.1, RIBBON1.MP1, RIBBON1.MP2; no longer FRAM.7, H2.MOUNT, POWER.2, RIBBON.14, RIBBON.MP1, RIBBON.MP2, SERIAL.4
- net LEDDATA: now also FACEBOARD.7, RIBBON1.7; no longer RIBBON.8
- net RST: now also RESET.1; no longer POWER.3, SERIAL.5, U$1.RST
- net VIN: now also J1.1; no longer H1.MOUNT, POWER.1
- net VUSB: no longer POWER.4

Commit message: tidy routing
Connections:
- removed net VIN: J1.1, U$1.RAW
- net 5V: now also J1.1, U$1.RAW
Changed lines of the file:
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@@
-</segment>
-</net>
-<net name="VIN" class="0">
-<segment>
-<pinref part="U$1" gate="G$1" pin="RAW"/>
-<wire x1="38.1" y1="38.1" x2="2.54" y2="38.1" width="0.1524" layer="91"/>
-<label x="-7.62" y="38.1" size="1.778" layer="95" rot="R180" xref="yes"/>
-</segment>
-<segment>
-<pinref part="J1" gate="G$1" pin="1"/>
-<wire x1="15.24" y1="22.86" x2="17.78" y2="22.86" width="0.1524" layer="91"/>
-<label x="17.78" y="22.86" size="1.778" layer="95" xref="yes"/>
 </segment>
 </net>
@@
 <pinref part="FACEBOARD" gate="G$1" pin="3"/>
 </segment>
+<segment>
+<pinref part="U$1" gate="G$1" pin="RAW"/>
+<wire x1="38.1" y1="38.1" x2="2.54" y2="38.1" width="0.1524" layer="91"/>
+<label x="-7.62" y="38.1" size="1.778" layer="95" rot="R180" xref="yes"/>
+</segment>
+<segment>
+<pinref part="J1" gate="G$1" pin="1"/>
+<wire x1="15.24" y1="22.86" x2="17.78" y2="22.86" width="0.1524" layer="91"/>
+<label x="17.78" y="22.86" size="1.778" layer="95" xref="yes"/>
+</segment>
 </net>
