File: faceboard-7-sensor/controller-board.brd (EAGLE design)
At the start: 36.7 x 60.6 mm, 7 parts, among them J1 DCJ0202

Commit message: redraw schematics
Parts:
- SV2: value FACEBOARDS -> SENSOR_BOARD
Connections:
- net FRAM_CLK renamed CLK
- net FRAM_CS renamed CS
- net FRAM_MISO renamed MISO
- net FRAM_MOSI renamed MOSI
- net LEDDATA renamed DIN
- net ROTA renamed RA
- net ROTB renamed RB
- net ROTC renamed RC
- net VIN renamed VCC
- removed net AREF: U$1.AREF
- removed net D0: U$1.TX0
- removed net D1: U$1.RX1
- removed net D13: U$1.D13
- removed net N$3: FRAM.6
- removed net N$8: FRAM.1
- removed net VUSB: U$1.5V
- net A0: now also ANALOG.1; no longer ANALOG.8
- net A1: now also ANALOG.2; no longer ANALOG.7
- net A2: now also ANALOG.3; no longer ANALOG.6
- net A3: now also ANALOG.4; no longer ANALOG.5
- net A4: now also ANALOG.5; no longer ANALOG.4
- net A5: now also ANALOG.6; no longer ANALOG.3
- net A6: now also ANALOG.7; no longer ANALOG.2
- net A7: now also ANALOG.8; no longer ANALOG.1
- net GND: no longer U$1.GND
- net RST: no longer U$1.RST1
Routing:
- net VCC: track 28.9 -> 0.05 mm
- net A7: track 4.08 -> 18.2 mm
- net A0: track 4.08 -> 18.2 mm
- net A6: track 4.08 -> 13.3 mm
- net A1: track 4.08 -> 13.3 mm
- net RST: track 47.7 -> 39.3 mm
- net A5: track 4.08 -> 8.64 mm
- net A2: track 4.08 -> 8.64 mm
- net A4: track 4.08 -> 4.81 mm
- net A3: track 4.08 -> 4.81 mm
Changed lines of the file:
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@@
 </autorouter>
 <elements>
-<element name="SV2" library="con-lstb" library_urn="urn:adsk.eagle:library:162" package="MA08-1" package3d_urn="urn:adsk.eagle:package:8343/1" value="FACEBOARDS" x="3.302" y="24.003" smashed="yes" rot="R270">
+<element name="SV2" library="con-lstb" library_urn="urn:adsk.eagle:library:162" package="MA08-1" package3d_urn="urn:adsk.eagle:package:8343/1" value="SENSOR_BOARD" x="3.302" y="24.003" smashed="yes" rot="R270">
 <attribute name="MF" value="" x="-56.388" y="-20.447" size="1.778" layer="27" rot="R270" display="off"/>
 <attribute name="MPN" value="" x="-56.388" y="-20.447" size="1.778" layer="27" rot="R270" display="off"/>
@@
 <signal name="RST">
 <contactref element="U$1" pad="RST"/>
-<contactref element="U$1" pad="RST1"/>
 <contactref element="RESET" pad="2"/>
-<wire x1="9.002" y1="32.893" x2="4.619" y2="37.276" width="0.1524" layer="1"/>
 <wire x1="4.619" y1="37.276" x2="4.619" y2="38.5150875" width="0.1524" layer="1"/>
 <wire x1="3.73" y1="39.4040875" x2="3.73" y2="39.76" width="0.1524" layer="1"/>
@@
 <wire x1="7.9824125" y1="28.6956" x2="7.4654" y2="28.1785875" width="0.1524" layer="16"/>
 <wire x1="7.4654" y1="19.8274125" x2="7.9824125" y2="19.3104" width="0.1524" layer="16"/>
-<wire x1="9.002" y1="32.893" x2="10.5386" y2="31.3564" width="0.1524" layer="16"/>
 <wire x1="10.5386" y1="31.3564" x2="10.5386" y2="29.9874125" width="0.1524" layer="16"/>
 <wire x1="10.5386" y1="29.9874125" x2="9.2467875" y2="28.6956" width="0.1524" layer="16"/>
@@
 <wire x1="7.9824125" y1="19.3104" x2="11.22243125" y2="19.3104" width="0.1524" layer="16"/>
 <wire x1="11.22243125" y1="19.3104" x2="19.7142" y2="27.80216875" width="0.1524" layer="16"/>
-</signal>
-<signal name="VIN">
-<contactref element="SV2" pad="2"/>
-<contactref element="U$1" pad="RAW"/>
-<contactref element="J1" pad="1"/>
-<wire x1="28.002" y1="38.011" x2="27.964" y2="37.973" width="1.27" layer="1"/>
-<wire x1="27.964" y1="37.973" x2="24.242" y2="37.973" width="1.27" layer="1"/>
-<wire x1="5.3848" y1="32.34590625" x2="4.61109375" y2="31.5722" width="0.8128" layer="16"/>
-<wire x1="4.61109375" y1="31.5722" x2="4.5212" y2="31.5722" width="0.8128" layer="16"/>
-<wire x1="4.5212" y1="31.5722" x2="3.302" y2="30.353" width="0.8128" layer="16"/>
-<wire x1="24.242" y1="37.973" x2="11.3711625" y2="37.973" width="0.8128" layer="16"/>
-<wire x1="11.3711625" y1="37.973" x2="10.0439625" y2="36.6458" width="0.8128" layer="16"/>
-<wire x1="10.0439625" y1="36.6458" x2="7.8456375" y2="36.6458" width="0.8128" layer="16"/>
-<wire x1="7.8456375" y1="36.6458" x2="5.3848" y2="34.1849625" width="0.8128" layer="16"/>
-<wire x1="5.3848" y1="34.1849625" x2="5.3848" y2="32.34590625" width="0.8128" layer="16"/>
+<wire x1="10.5386" y1="31.3564" x2="4.619" y2="37.276" width="0" layer="19" extent="1-16"/>
 </signal>
 <signal name="GND">
@@
 <contactref element="FRAM" pad="7"/>
 <contactref element="ROTARY" pad="4"/>
-<contactref element="U$1" pad="GND"/>
 <contactref element="J1" pad="2"/>
 <contactref element="J1" pad="3"/>
 <contactref element="U$1" pad="GND1"/>
 <contactref element="RESET" pad="1"/>
-</signal>
-<signal name="LEDDATA">
-<contactref element="U$1" pad="D9"/>
-<contactref element="SV2" pad="7"/>
-<wire x1="9.002" y1="10.033" x2="5.08" y2="13.955" width="0.2032" layer="16"/>
-<wire x1="3.302" y1="17.31184375" x2="3.302" y2="17.653" width="0.2032" layer="16"/>
-<wire x1="5.08" y1="13.955" x2="5.08" y2="15.53384375" width="0.2032" layer="16"/>
-<wire x1="5.08" y1="15.53384375" x2="3.302" y2="17.31184375" width="0.2032" layer="16"/>
-</signal>
-<signal name="FRAM_CS">
+<wire x1="34.102" y1="38.011" x2="31.102" y2="42.811" width="0" layer="19" extent="1-1"/>
+<wire x1="9.002" y1="30.353" x2="31.102" y2="42.811" width="0" layer="19" extent="1-1"/>
+<wire x1="3.302" y1="32.893" x2="9.002" y2="30.353" width="0" layer="19" extent="1-1"/>
+<wire x1="3.73" y1="37.76" x2="3.302" y2="32.893" width="0" layer="19" extent="1-1"/>
+<wire x1="4.875" y1="48.498" x2="3.73" y2="37.76" width="0" layer="19" extent="1-1"/>
+<wire x1="3.2037125" y1="9" x2="9.002" y2="30.353" width="0" layer="19" extent="1-1"/>
+</signal>
+<signal name="CS">
 <contactref element="FRAM" pad="2"/>
 <contactref element="U$1" pad="D2"/>
@@
 <wire x1="15.34116875" y1="32.1752" x2="10.97896875" y2="27.813" width="0.1524" layer="1"/>
 </signal>
-<signal name="FRAM_MOSI">
+<signal name="MOSI">
 <contactref element="FRAM" pad="3"/>
 <contactref element="U$1" pad="D3"/>
@@
 <wire x1="1.5494" y1="29.5656" x2="3.302" y2="27.813" width="0.1524" layer="16"/>
 </signal>
-<signal name="FRAM_CLK">
+<signal name="CLK">
 <contactref element="FRAM" pad="5"/>
 <contactref element="U$1" pad="D5"/>
@@
 <wire x1="18.3274" y1="40.1256" x2="9.955" y2="48.498" width="0.1524" layer="16"/>
 </signal>
-<signal name="FRAM_MISO">
+<signal name="MISO">
 <contactref element="FRAM" pad="4"/>
 <contactref element="U$1" pad="D4"/>
@@
 <wire x1="22" y1="28.56894375" x2="18.39925625" y2="24.9682" width="0.1524" layer="1"/>
 </signal>
-<signal name="N$3">
-<contactref element="FRAM" pad="6"/>
-</signal>
-<signal name="N$8">
-<contactref element="FRAM" pad="1"/>
-</signal>
-<signal name="ROTA">
+<signal name="RA">
 <contactref element="ROTARY" pad="3"/>
 <contactref element="U$1" pad="D10"/>
@@
 <wire x1="8.509" y1="7" x2="9.002" y2="7.493" width="0.8128" layer="1"/>
 </signal>
-<signal name="ROTC">
+<signal name="RC">
 <contactref element="ROTARY" pad="1"/>
 <contactref element="U$1" pad="D12"/>
@@
 <wire x1="3.7907125" y1="2.413" x2="9.002" y2="2.413" width="0.8128" layer="1"/>
 </signal>
-<signal name="ROTB">
+<signal name="RB">
 <contactref element="ROTARY" pad="2"/>
 <contactref element="U$1" pad="D11"/>
@@
 </signal>
 <signal name="A7">
+<contactref element="U$1" pad="A7"/>
+<wire x1="28.322" y1="10.033" x2="24.242" y2="27.813" width="0.8128" layer="1"/>
+<contactref element="ANALOG" pad="8"/>
+</signal>
+<signal name="A6">
+<contactref element="U$1" pad="A6"/>
+<wire x1="28.322" y1="12.573" x2="24.242" y2="25.273" width="0.8128" layer="1"/>
+<contactref element="ANALOG" pad="7"/>
+</signal>
+<signal name="A5">
+<contactref element="U$1" pad="A5"/>
+<wire x1="28.322" y1="15.113" x2="24.242" y2="22.733" width="0.8128" layer="1"/>
+<contactref element="ANALOG" pad="6"/>
+</signal>
+<signal name="A4">
+<contactref element="U$1" pad="A4"/>
+<wire x1="28.322" y1="17.653" x2="24.242" y2="20.193" width="0.8128" layer="1"/>
+<contactref element="ANALOG" pad="5"/>
+</signal>
+<signal name="A3">
+<contactref element="U$1" pad="A3"/>
+<wire x1="28.322" y1="20.193" x2="24.242" y2="17.653" width="0.8128" layer="1"/>
+<contactref element="ANALOG" pad="4"/>
+</signal>
+<signal name="A2">
+<contactref element="U$1" pad="A2"/>
+<wire x1="28.322" y1="22.733" x2="24.242" y2="15.113" width="0.8128" layer="1"/>
+<contactref element="ANALOG" pad="3"/>
+</signal>
+<signal name="A1">
+<contactref element="U$1" pad="A1"/>
+<wire x1="28.322" y1="25.273" x2="24.242" y2="12.573" width="0.8128" layer="1"/>
+<contactref element="ANALOG" pad="2"/>
+</signal>
+<signal name="A0">
+<contactref element="U$1" pad="A0"/>
+<wire x1="28.322" y1="27.813" x2="24.242" y2="10.033" width="0.8128" layer="1"/>
 <contactref element="ANALOG" pad="1"/>
-<contactref element="U$1" pad="A7"/>
-<wire x1="28.322" y1="27.813" x2="24.242" y2="27.813" width="0.8128" layer="1"/>
-</signal>
-<signal name="A6">
-<contactref element="ANALOG" pad="2"/>
-<contactref element="U$1" pad="A6"/>
-<wire x1="28.322" y1="25.273" x2="24.242" y2="25.273" width="0.8128" layer="1"/>
-</signal>
-<signal name="A5">
-<contactref element="ANALOG" pad="3"/>
-<contactref element="U$1" pad="A5"/>
-<wire x1="28.322" y1="22.733" x2="24.242" y2="22.733" width="0.8128" layer="1"/>
-</signal>
-<signal name="A4">
-<contactref element="ANALOG" pad="4"/>
-<contactref element="U$1" pad="A4"/>
-<wire x1="28.322" y1="20.193" x2="24.242" y2="20.193" width="0.8128" layer="1"/>
-</signal>
-<signal name="A3">
-<contactref element="ANALOG" pad="5"/>
-<contactref element="U$1" pad="A3"/>
-<wire x1="28.322" y1="17.653" x2="24.242" y2="17.653" width="0.8128" layer="1"/>
-</signal>
-<signal name="A2">
-<contactref element="ANALOG" pad="6"/>
-<contactref element="U$1" pad="A2"/>
-<wire x1="28.322" y1="15.113" x2="24.242" y2="15.113" width="0.8128" layer="1"/>
-</signal>
-<signal name="A1">
-<contactref element="ANALOG" pad="7"/>
-<contactref element="U$1" pad="A1"/>
-<wire x1="28.322" y1="12.573" x2="24.242" y2="12.573" width="0.8128" layer="1"/>
-</signal>
-<signal name="A0">
-<contactref element="ANALOG" pad="8"/>
-<contactref element="U$1" pad="A0"/>
-<wire x1="28.322" y1="10.033" x2="24.242" y2="10.033" width="0.8128" layer="1"/>
-</signal>
-<signal name="VUSB">
-<contactref element="U$1" pad="5V"/>
-</signal>
-<signal name="D13">
-<contactref element="U$1" pad="D13"/>
-</signal>
-<signal name="AREF">
-<contactref element="U$1" pad="AREF"/>
-</signal>
-<signal name="D0">
-<contactref element="U$1" pad="TX0"/>
-</signal>
-<signal name="D1">
-<contactref element="U$1" pad="RX1"/>
+</signal>
+<signal name="DIN">
+<contactref element="SV2" pad="7"/>
+<contactref element="U$1" pad="D9"/>
+<wire x1="9.002" y1="10.033" x2="5.08" y2="13.955" width="0.2032" layer="16"/>
+<wire x1="5.08" y1="13.955" x2="5.08" y2="15.53384375" width="0.2032" layer="16"/>
+<wire x1="5.08" y1="15.53384375" x2="3.302" y2="17.31184375" width="0.2032" layer="16"/>
+<wire x1="3.302" y1="17.31184375" x2="3.302" y2="17.653" width="0" layer="19" extent="16-16"/>
+</signal>
+<signal name="VCC">
+<contactref element="SV2" pad="2"/>
+<contactref element="J1" pad="1"/>
+<wire x1="28.002" y1="38.011" x2="27.964" y2="37.973" width="1.27" layer="1"/>
+<contactref element="U$1" pad="RAW"/>
+<wire x1="24.242" y1="37.973" x2="27.964" y2="37.973" width="0" layer="19" extent="1-1"/>
+<wire x1="3.302" y1="30.353" x2="24.242" y2="37.973" width="0" layer="19" extent="1-1"/>
 </signal>
 </signals>

Commit message: reroute
Parts:
- turned ANALOG to 90 degrees
Routing:
- net VCC: track 0.05 -> 40.0 mm, vias 0 -> 2
- net A7: track 18.2 -> 4.08 mm
- net A0: track 18.2 -> 4.08 mm
- net A6: track 13.3 -> 4.08 mm
- net A1: track 13.3 -> 4.08 mm
- net RST: track 39.3 -> 44.4 mm
- net A5: track 8.64 -> 4.08 mm
- net A2: track 8.64 -> 4.08 mm
- net A4: track 4.81 -> 4.08 mm
- net A3: track 4.81 -> 4.08 mm
Other:
- board text added: "Nemus Controller Board v0.1.2"
- board text removed: "Nemus Controller Board v0.1.1"
Changed lines of the file:
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@@
 <rectangle x1="27.9287" y1="49.903809375" x2="28.3974" y2="49.981940625" layer="200" rot="R180"/>
 <rectangle x1="26.2099" y1="49.903809375" x2="26.3662" y2="49.981940625" layer="200" rot="R180"/>
-<text x="33.248" y="19.2" size="1.016" layer="21" ratio="15" rot="R90" align="center">Nemus Controller Board v0.1.1</text>
+<text x="33.248" y="19.2" size="1.016" layer="21" ratio="15" rot="R90" align="center">Nemus Controller Board v0.1.2</text>
 <rectangle x1="-0.000509375" y1="-0.000509375" x2="0.129540625" y2="0.000509375" layer="202"/>
 <rectangle x1="-0.000509375" y1="0.000509375" x2="0.129540625" y2="0.001525" layer="202"/>
@@
 <attribute name="NAME" x="5.649728125" y="3.91846875" size="1.016" layer="25" ratio="18" rot="R90"/>
 </element>
-<element name="ANALOG" library="con-lstb" library_urn="urn:adsk.eagle:library:162" package="MA08-1" package3d_urn="urn:adsk.eagle:package:8343/1" value="SIGNALS" x="28.322" y="18.923" smashed="yes" rot="R270">
-<attribute name="MF" value="" x="38.482" y="18.923" size="1.778" layer="27" rot="R270" display="off"/>
-<attribute name="MPN" value="" x="38.482" y="18.923" size="1.778" layer="27" rot="R270" display="off"/>
-<attribute name="NAME" x="30.227" y="28.829" size="1.27" layer="25" ratio="10" rot="R270"/>
-<attribute name="OC_FARNELL" value="unknown" x="38.482" y="18.923" size="1.778" layer="27" rot="R270" display="off"/>
-<attribute name="OC_NEWARK" value="unknown" x="38.482" y="18.923" size="1.778" layer="27" rot="R270" display="off"/>
-<attribute name="POPULARITY" value="10" x="38.482" y="18.923" size="1.778" layer="27" rot="R270" display="off"/>
-<attribute name="VALUE" x="30.354" y="18.415" size="1.27" layer="27" ratio="10" rot="R270"/>
+<element name="ANALOG" library="con-lstb" library_urn="urn:adsk.eagle:library:162" package="MA08-1" package3d_urn="urn:adsk.eagle:package:8343/1" value="SIGNALS" x="28.322" y="18.923" smashed="yes" rot="R90">
+<attribute name="MF" value="" x="18.162" y="18.923" size="1.778" layer="27" rot="R90" display="off"/>
+<attribute name="MPN" value="" x="18.162" y="18.923" size="1.778" layer="27" rot="R90" display="off"/>
+<attribute name="NAME" x="26.417" y="9.017" size="1.27" layer="25" ratio="10" rot="R90"/>
+<attribute name="OC_FARNELL" value="unknown" x="18.162" y="18.923" size="1.778" layer="27" rot="R90" display="off"/>
+<attribute name="OC_NEWARK" value="unknown" x="18.162" y="18.923" size="1.778" layer="27" rot="R90" display="off"/>
+<attribute name="POPULARITY" value="10" x="18.162" y="18.923" size="1.778" layer="27" rot="R90" display="off"/>
+<attribute name="VALUE" x="26.29" y="19.431" size="1.27" layer="27" ratio="10" rot="R90"/>
 </element>
 <element name="J1" library="con-jack" library_urn="urn:adsk.eagle:library:154" package="DCJ0202" package3d_urn="urn:adsk.eagle:package:7491/1" value="DCJ0202" x="31.102" y="38.011" smashed="yes" rot="R90">
@@
 <contactref element="U$1" pad="RST"/>
 <contactref element="RESET" pad="2"/>
-<wire x1="4.619" y1="37.276" x2="4.619" y2="38.5150875" width="0.1524" layer="1"/>
-<wire x1="3.73" y1="39.4040875" x2="3.73" y2="39.76" width="0.1524" layer="1"/>
-<wire x1="4.619" y1="38.5150875" x2="3.73" y2="39.4040875" width="0.1524" layer="1"/>
-<wire x1="7.9824125" y1="28.6956" x2="7.4654" y2="28.1785875" width="0.1524" layer="16"/>
-<wire x1="7.4654" y1="19.8274125" x2="7.9824125" y2="19.3104" width="0.1524" layer="16"/>
-<wire x1="10.5386" y1="31.3564" x2="10.5386" y2="29.9874125" width="0.1524" layer="16"/>
-<wire x1="10.5386" y1="29.9874125" x2="9.2467875" y2="28.6956" width="0.1524" layer="16"/>
-<wire x1="9.2467875" y1="28.6956" x2="7.9824125" y2="28.6956" width="0.1524" layer="16"/>
+<wire x1="7.9824125" y1="19.3104" x2="7.4654" y2="19.8274125" width="0.1524" layer="16"/>
 <wire x1="19.7142" y1="27.80216875" x2="19.7142" y2="28.3652" width="0.1524" layer="16"/>
 <wire x1="19.7142" y1="28.3652" x2="24.242" y2="32.893" width="0.1524" layer="16"/>
-<wire x1="7.4654" y1="28.1785875" x2="7.4654" y2="19.8274125" width="0.1524" layer="16"/>
 <wire x1="7.9824125" y1="19.3104" x2="11.22243125" y2="19.3104" width="0.1524" layer="16"/>
 <wire x1="11.22243125" y1="19.3104" x2="19.7142" y2="27.80216875" width="0.1524" layer="16"/>
-<wire x1="10.5386" y1="31.3564" x2="4.619" y2="37.276" width="0" layer="19" extent="1-16"/>
+<wire x1="7.4654" y1="19.8274125" x2="7.4654" y2="36.0246" width="0.1524" layer="16"/>
+<wire x1="7.4654" y1="36.0246" x2="3.73" y2="39.76" width="0.1524" layer="16"/>
 </signal>
 <signal name="GND">
@@
 <contactref element="U$1" pad="GND1"/>
 <contactref element="RESET" pad="1"/>
-<wire x1="34.102" y1="38.011" x2="31.102" y2="42.811" width="0" layer="19" extent="1-1"/>
-<wire x1="9.002" y1="30.353" x2="31.102" y2="42.811" width="0" layer="19" extent="1-1"/>
-<wire x1="3.302" y1="32.893" x2="9.002" y2="30.353" width="0" layer="19" extent="1-1"/>
-<wire x1="3.73" y1="37.76" x2="3.302" y2="32.893" width="0" layer="19" extent="1-1"/>
-<wire x1="4.875" y1="48.498" x2="3.73" y2="37.76" width="0" layer="19" extent="1-1"/>
-<wire x1="3.2037125" y1="9" x2="9.002" y2="30.353" width="0" layer="19" extent="1-1"/>
 </signal>
 <signal name="CS">
@@
 <signal name="A7">
 <contactref element="U$1" pad="A7"/>
-<wire x1="28.322" y1="10.033" x2="24.242" y2="27.813" width="0.8128" layer="1"/>
+<wire x1="28.322" y1="27.813" x2="24.242" y2="27.813" width="0.8128" layer="1"/>
 <contactref element="ANALOG" pad="8"/>
 </signal>
 <signal name="A6">
 <contactref element="U$1" pad="A6"/>
-<wire x1="28.322" y1="12.573" x2="24.242" y2="25.273" width="0.8128" layer="1"/>
+<wire x1="28.322" y1="25.273" x2="24.242" y2="25.273" width="0.8128" layer="1"/>
 <contactref element="ANALOG" pad="7"/>
 </signal>
 <signal name="A5">
 <contactref element="U$1" pad="A5"/>
-<wire x1="28.322" y1="15.113" x2="24.242" y2="22.733" width="0.8128" layer="1"/>
+<wire x1="28.322" y1="22.733" x2="24.242" y2="22.733" width="0.8128" layer="1"/>
 <contactref element="ANALOG" pad="6"/>
 </signal>
 <signal name="A4">
 <contactref element="U$1" pad="A4"/>
-<wire x1="28.322" y1="17.653" x2="24.242" y2="20.193" width="0.8128" layer="1"/>
+<wire x1="28.322" y1="20.193" x2="24.242" y2="20.193" width="0.8128" layer="1"/>
 <contactref element="ANALOG" pad="5"/>
 </signal>
 <signal name="A3">
 <contactref element="U$1" pad="A3"/>
-<wire x1="28.322" y1="20.193" x2="24.242" y2="17.653" width="0.8128" layer="1"/>
+<wire x1="28.322" y1="17.653" x2="24.242" y2="17.653" width="0.8128" layer="1"/>
 <contactref element="ANALOG" pad="4"/>
 </signal>
 <signal name="A2">
 <contactref element="U$1" pad="A2"/>
-<wire x1="28.322" y1="22.733" x2="24.242" y2="15.113" width="0.8128" layer="1"/>
+<wire x1="28.322" y1="15.113" x2="24.242" y2="15.113" width="0.8128" layer="1"/>
 <contactref element="ANALOG" pad="3"/>
 </signal>
 <signal name="A1">
 <contactref element="U$1" pad="A1"/>
-<wire x1="28.322" y1="25.273" x2="24.242" y2="12.573" width="0.8128" layer="1"/>
+<wire x1="28.322" y1="12.573" x2="24.242" y2="12.573" width="0.8128" layer="1"/>
 <contactref element="ANALOG" pad="2"/>
 </signal>
 <signal name="A0">
 <contactref element="U$1" pad="A0"/>
-<wire x1="28.322" y1="27.813" x2="24.242" y2="10.033" width="0.8128" layer="1"/>
+<wire x1="28.322" y1="10.033" x2="24.242" y2="10.033" width="0.8128" layer="1"/>
 <contactref element="ANALOG" pad="1"/>
 </signal>
@@
 <wire x1="9.002" y1="10.033" x2="5.08" y2="13.955" width="0.2032" layer="16"/>
 <wire x1="5.08" y1="13.955" x2="5.08" y2="15.53384375" width="0.2032" layer="16"/>
-<wire x1="5.08" y1="15.53384375" x2="3.302" y2="17.31184375" width="0.2032" layer="16"/>
-<wire x1="3.302" y1="17.31184375" x2="3.302" y2="17.653" width="0" layer="19" extent="16-16"/>
+<wire x1="3.302" y1="17.31184375" x2="5.08" y2="15.53384375" width="0.2032" layer="16"/>
+<wire x1="3.302" y1="17.653" x2="3.302" y2="17.31184375" width="0.2" layer="16"/>
 </signal>
 <signal name="VCC">
 <contactref element="SV2" pad="2"/>
 <contactref element="J1" pad="1"/>
+<contactref element="U$1" pad="RAW"/>
 <wire x1="28.002" y1="38.011" x2="27.964" y2="37.973" width="1.27" layer="1"/>
-<contactref element="U$1" pad="RAW"/>
-<wire x1="24.242" y1="37.973" x2="27.964" y2="37.973" width="0" layer="19" extent="1-1"/>
-<wire x1="3.302" y1="30.353" x2="24.242" y2="37.973" width="0" layer="19" extent="1-1"/>
+<wire x1="27.964" y1="37.973" x2="24.242" y2="37.973" width="1.27" layer="1"/>
+<via x="16" y="45" extent="1-16" drill="0.35"/>
+<wire x1="3.302" y1="30.353" x2="4.2926" y2="31.3436" width="1.27" layer="1"/>
+<wire x1="4.2926" y1="31.3436" x2="4.7057875" y2="31.3436" width="1.27" layer="1"/>
+<wire x1="6.9066" y1="38.57005" x2="7.75095" y2="39.4144" width="1.27" layer="1"/>
+<wire x1="4.7057875" y1="31.3436" x2="6.9066" y2="33.5444125" width="1.27" layer="1"/>
+<wire x1="6.9066" y1="33.5444125" x2="6.9066" y2="38.57005" width="1.27" layer="1"/>
+<wire x1="7.75095" y1="39.4144" x2="10.4144" y2="39.4144" width="1.27" layer="1"/>
+<wire x1="10.4144" y1="39.4144" x2="16" y2="45" width="1.27" layer="1"/>
+<wire x1="16" y1="45" x2="23" y2="45" width="1.27" layer="16"/>
+<via x="23" y="45" extent="1-16" drill="0.35"/>
+<wire x1="23" y1="45" x2="24.242" y2="43.758" width="1.27" layer="1"/>
+<wire x1="24.242" y1="43.758" x2="24.242" y2="37.973" width="1.27" layer="1"/>
 </signal>
 </signals>
