File: faceboard-3-sensor/double-wired-3-face-board.brd (EAGLE design)
At the start: 14 x 51 mm, 14 parts, among them Q1 QRE1113, Q2 QRE1113, Q3 QRE1113, Q4 QRE1113, Q5 QRE1113, Q6 QRE1113

Commit message: tidy
Parts:
- R2, R4, R6: value 10k -> 100k
Connections:
- net N$1 renamed 5VQ1
- net N$3 renamed 5VQ2
- net N$5 renamed 5VQ3
Routing:
- net VCC: track 47.4 -> 44.0 mm
- net S1: track 64.9 -> 62.6 mm
