File: faceboard-3-sensor/double-wired-3-face-board.sch (EAGLE design)
At the start: 14 parts, among them Q1 QRE1113, Q2 QRE1113, Q3 QRE1113, Q4 QRE1113, Q5 QRE1113, Q6 QRE1113

Commit message: re-draw schematics
Changed lines of the file:
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@@
 <layers>
 <layer number="1" name="Top" color="4" fill="1" visible="no" active="no"/>
+<layer number="2" name="Route2" color="1" fill="3" visible="no" active="no"/>
+<layer number="3" name="Route3" color="4" fill="3" visible="no" active="no"/>
+<layer number="4" name="Route4" color="1" fill="4" visible="no" active="no"/>
+<layer number="5" name="Route5" color="4" fill="4" visible="no" active="no"/>
+<layer number="6" name="Route6" color="1" fill="8" visible="no" active="no"/>
+<layer number="7" name="Route7" color="4" fill="8" visible="no" active="no"/>
+<layer number="8" name="Route8" color="1" fill="2" visible="no" active="no"/>
+<layer number="9" name="Route9" color="4" fill="2" visible="no" active="no"/>
+<layer number="10" name="Route10" color="1" fill="7" visible="no" active="no"/>
+<layer number="11" name="Route11" color="4" fill="7" visible="no" active="no"/>
+<layer number="12" name="Route12" color="1" fill="5" visible="no" active="no"/>
+<layer number="13" name="Route13" color="4" fill="5" visible="no" active="no"/>
+<layer number="14" name="Route14" color="1" fill="6" visible="no" active="no"/>
+<layer number="15" name="Route15" color="4" fill="6" visible="no" active="no"/>
 <layer number="16" name="Bottom" color="1" fill="1" visible="no" active="no"/>
 <layer number="17" name="Pads" color="2" fill="1" visible="no" active="no"/>
@@
 <pinref part="Q1" gate="A" pin="1"/>
 <pinref part="R1" gate="G$1" pin="2"/>
-<wire x1="12.7" y1="81.28" x2="12.7" y2="76.2" width="0.1524" layer="91"/>
-<junction x="12.7" y="81.28"/>
+<wire x1="15.24" y1="78.74" x2="12.7" y2="76.2" width="0.1524" layer="91"/>
+<junction x="15.24" y="78.74"/>
 <wire x1="12.7" y1="76.2" x2="5.08" y2="76.2" width="0.1524" layer="91"/>
 <pinref part="Q4" gate="A" pin="1"/>
 <wire x1="5.08" y1="76.2" x2="5.08" y2="38.1" width="0.1524" layer="91"/>
-<wire x1="5.08" y1="38.1" x2="12.7" y2="38.1" width="0.1524" layer="91"/>
+<wire x1="5.08" y1="38.1" x2="15.24" y2="35.56" width="0.1524" layer="91"/>
+<wire x1="12.7" y1="81.28" x2="15.24" y2="78.74" width="0.1524" layer="91"/>
 </segment>
 </net>
@@
 <pinref part="Q1" gate="A" pin="3"/>
 <pinref part="R2" gate="G$1" pin="1"/>
-<wire x1="53.34" y1="83.82" x2="50.8" y2="83.82" width="0.1524" layer="91"/>
+<wire x1="53.34" y1="83.82" x2="30.48" y2="78.74" width="0.1524" layer="91"/>
 <pinref part="Q4" gate="A" pin="3"/>
 <wire x1="53.34" y1="83.82" x2="53.34" y2="53.34" width="0.1524" layer="91"/>
 <wire x1="53.34" y1="53.34" x2="53.34" y2="40.64" width="0.1524" layer="91"/>
-<wire x1="53.34" y1="40.64" x2="50.8" y2="40.64" width="0.1524" layer="91"/>
+<wire x1="53.34" y1="40.64" x2="30.48" y2="35.56" width="0.1524" layer="91"/>
 <junction x="53.34" y="83.82"/>
 <wire x1="53.34" y1="53.34" x2="58.42" y2="53.34" width="0.1524" layer="91"/>
 <junction x="53.34" y="53.34"/>
-<label x="58.42" y="53.34" size="1.778" layer="95" xref="yes"/>
+<label x="63.754" y="53.34" size="1.778" layer="95" rot="R180" xref="yes"/>
 </segment>
 <segment>
@@
 <pinref part="Q1" gate="A" pin="2"/>
 <pinref part="GND1" gate="1" pin="GND"/>
-<wire x1="12.7" y1="73.66" x2="12.7" y2="60.96" width="0.1524" layer="91"/>
+<wire x1="15.24" y1="76.2" x2="12.7" y2="60.96" width="0.1524" layer="91"/>
 <wire x1="12.7" y1="60.96" x2="30.48" y2="60.96" width="0.1524" layer="91"/>
 <pinref part="Q1" gate="A" pin="4"/>
-<wire x1="50.8" y1="68.58" x2="50.8" y2="60.96" width="0.1524" layer="91"/>
+<wire x1="30.48" y1="76.2" x2="50.8" y2="60.96" width="0.1524" layer="91"/>
 <wire x1="50.8" y1="60.96" x2="30.48" y2="60.96" width="0.1524" layer="91"/>
 <junction x="30.48" y="60.96"/>
@@
 <pinref part="Q2" gate="A" pin="2"/>
 <pinref part="GND2" gate="1" pin="GND"/>
-<wire x1="76.2" y1="73.66" x2="76.2" y2="60.96" width="0.1524" layer="91"/>
+<wire x1="78.74" y1="76.2" x2="76.2" y2="60.96" width="0.1524" layer="91"/>
 <wire x1="76.2" y1="60.96" x2="93.98" y2="60.96" width="0.1524" layer="91"/>
 <pinref part="Q2" gate="A" pin="4"/>
-<wire x1="114.3" y1="68.58" x2="114.3" y2="60.96" width="0.1524" layer="91"/>
+<wire x1="93.98" y1="76.2" x2="114.3" y2="60.96" width="0.1524" layer="91"/>
 <wire x1="114.3" y1="60.96" x2="93.98" y2="60.96" width="0.1524" layer="91"/>
 <junction x="93.98" y="60.96"/>
@@
 <pinref part="Q3" gate="A" pin="2"/>
 <pinref part="GND3" gate="1" pin="GND"/>
-<wire x1="142.24" y1="73.66" x2="142.24" y2="60.96" width="0.1524" layer="91"/>
+<wire x1="144.78" y1="76.2" x2="142.24" y2="60.96" width="0.1524" layer="91"/>
 <wire x1="142.24" y1="60.96" x2="160.02" y2="60.96" width="0.1524" layer="91"/>
 <pinref part="Q3" gate="A" pin="4"/>
-<wire x1="180.34" y1="68.58" x2="180.34" y2="60.96" width="0.1524" layer="91"/>
+<wire x1="160.02" y1="76.2" x2="180.34" y2="60.96" width="0.1524" layer="91"/>
 <wire x1="180.34" y1="60.96" x2="160.02" y2="60.96" width="0.1524" layer="91"/>
 <junction x="160.02" y="60.96"/>
@@
 <pinref part="Q4" gate="A" pin="2"/>
 <pinref part="GND4" gate="1" pin="GND"/>
-<wire x1="12.7" y1="30.48" x2="12.7" y2="15.24" width="0.1524" layer="91"/>
+<wire x1="15.24" y1="33.02" x2="12.7" y2="15.24" width="0.1524" layer="91"/>
 <wire x1="12.7" y1="15.24" x2="30.48" y2="15.24" width="0.1524" layer="91"/>
 <pinref part="Q4" gate="A" pin="4"/>
-<wire x1="50.8" y1="25.4" x2="50.8" y2="15.24" width="0.1524" layer="91"/>
+<wire x1="30.48" y1="33.02" x2="50.8" y2="15.24" width="0.1524" layer="91"/>
 <wire x1="50.8" y1="15.24" x2="30.48" y2="15.24" width="0.1524" layer="91"/>
 <junction x="30.48" y="15.24"/>
@@
 <pinref part="Q5" gate="A" pin="2"/>
 <pinref part="GND5" gate="1" pin="GND"/>
-<wire x1="76.2" y1="30.48" x2="76.2" y2="15.24" width="0.1524" layer="91"/>
+<wire x1="78.74" y1="33.02" x2="76.2" y2="15.24" width="0.1524" layer="91"/>
 <wire x1="76.2" y1="15.24" x2="93.98" y2="15.24" width="0.1524" layer="91"/>
 <pinref part="Q5" gate="A" pin="4"/>
-<wire x1="114.3" y1="25.4" x2="114.3" y2="15.24" width="0.1524" layer="91"/>
+<wire x1="93.98" y1="33.02" x2="114.3" y2="15.24" width="0.1524" layer="91"/>
 <wire x1="114.3" y1="15.24" x2="93.98" y2="15.24" width="0.1524" layer="91"/>
 <junction x="93.98" y="15.24"/>
@@
 <pinref part="Q6" gate="A" pin="2"/>
 <pinref part="GND6" gate="1" pin="GND"/>
-<wire x1="142.24" y1="33.02" x2="142.24" y2="17.78" width="0.1524" layer="91"/>
+<wire x1="144.78" y1="35.56" x2="142.24" y2="17.78" width="0.1524" layer="91"/>
 <wire x1="142.24" y1="17.78" x2="162.56" y2="17.78" width="0.1524" layer="91"/>
 <pinref part="Q6" gate="A" pin="4"/>
-<wire x1="180.34" y1="27.94" x2="180.34" y2="17.78" width="0.1524" layer="91"/>
+<wire x1="160.02" y1="35.56" x2="180.34" y2="17.78" width="0.1524" layer="91"/>
 <wire x1="180.34" y1="17.78" x2="162.56" y2="17.78" width="0.1524" layer="91"/>
 <junction x="162.56" y="17.78"/>
@@
 <pinref part="SV2" gate="G$1" pin="1"/>
 <wire x1="-20.32" y1="50.8" x2="-15.24" y2="50.8" width="0.1524" layer="91"/>
-<label x="-15.24" y="50.8" size="1.778" layer="95" xref="yes"/>
+<label x="-7.62" y="50.8" size="1.778" layer="95" rot="R180" xref="yes"/>
 </segment>
 </net>
@@
 <pinref part="Q2" gate="A" pin="1"/>
 <pinref part="R3" gate="G$1" pin="2"/>
-<wire x1="76.2" y1="81.28" x2="76.2" y2="76.2" width="0.1524" layer="91"/>
+<wire x1="78.74" y1="78.74" x2="76.2" y2="76.2" width="0.1524" layer="91"/>
 <wire x1="76.2" y1="76.2" x2="73.66" y2="76.2" width="0.1524" layer="91"/>
-<junction x="76.2" y="81.28"/>
+<junction x="78.74" y="78.74"/>
 <pinref part="Q5" gate="A" pin="1"/>
 <wire x1="73.66" y1="76.2" x2="73.66" y2="38.1" width="0.1524" layer="91"/>
-<wire x1="73.66" y1="38.1" x2="76.2" y2="38.1" width="0.1524" layer="91"/>
+<wire x1="73.66" y1="38.1" x2="78.74" y2="35.56" width="0.1524" layer="91"/>
+<wire x1="76.2" y1="81.28" x2="78.74" y2="78.74" width="0.1524" layer="91"/>
 </segment>
 </net>
@@
 <pinref part="Q2" gate="A" pin="3"/>
 <pinref part="R4" gate="G$1" pin="1"/>
-<wire x1="116.84" y1="83.82" x2="114.3" y2="83.82" width="0.1524" layer="91"/>
+<wire x1="116.84" y1="83.82" x2="93.98" y2="78.74" width="0.1524" layer="91"/>
 <pinref part="Q5" gate="A" pin="3"/>
 <wire x1="116.84" y1="83.82" x2="116.84" y2="50.8" width="0.1524" layer="91"/>
 <wire x1="116.84" y1="50.8" x2="116.84" y2="40.64" width="0.1524" layer="91"/>
-<wire x1="116.84" y1="40.64" x2="114.3" y2="40.64" width="0.1524" layer="91"/>
+<wire x1="116.84" y1="40.64" x2="93.98" y2="35.56" width="0.1524" layer="91"/>
 <junction x="116.84" y="83.82"/>
 <wire x1="116.84" y1="50.8" x2="121.92" y2="50.8" width="0.1524" layer="91"/>
@@
 <pinref part="Q3" gate="A" pin="1"/>
 <pinref part="R5" gate="G$1" pin="2"/>
-<wire x1="142.24" y1="81.28" x2="142.24" y2="76.2" width="0.1524" layer="91"/>
+<wire x1="144.78" y1="78.74" x2="142.24" y2="76.2" width="0.1524" layer="91"/>
 <wire x1="142.24" y1="76.2" x2="139.7" y2="76.2" width="0.1524" layer="91"/>
-<junction x="142.24" y="81.28"/>
+<junction x="144.78" y="78.74"/>
 <pinref part="Q6" gate="A" pin="1"/>
 <wire x1="139.7" y1="76.2" x2="139.7" y2="40.64" width="0.1524" layer="91"/>
-<wire x1="139.7" y1="40.64" x2="142.24" y2="40.64" width="0.1524" layer="91"/>
+<wire x1="139.7" y1="40.64" x2="144.78" y2="38.1" width="0.1524" layer="91"/>
+<wire x1="142.24" y1="81.28" x2="144.78" y2="78.74" width="0.1524" layer="91"/>
 </segment>
 </net>
@@
 <pinref part="Q3" gate="A" pin="3"/>
 <pinref part="R6" gate="G$1" pin="1"/>
-<wire x1="182.88" y1="83.82" x2="180.34" y2="83.82" width="0.1524" layer="91"/>
+<wire x1="182.88" y1="83.82" x2="160.02" y2="78.74" width="0.1524" layer="91"/>
 <pinref part="Q6" gate="A" pin="3"/>
 <wire x1="182.88" y1="83.82" x2="182.88" y2="53.34" width="0.1524" layer="91"/>
 <wire x1="182.88" y1="53.34" x2="182.88" y2="43.18" width="0.1524" layer="91"/>
-<wire x1="182.88" y1="43.18" x2="180.34" y2="43.18" width="0.1524" layer="91"/>
+<wire x1="182.88" y1="43.18" x2="160.02" y2="38.1" width="0.1524" layer="91"/>
 <junction x="182.88" y="83.82"/>
 <wire x1="182.88" y1="53.34" x2="187.96" y2="53.34" width="0.1524" layer="91"/>

Commit message: tidy
Parts:
- R2, R4, R6: value 10k -> 100k
Connections:
- net N$1 renamed 5VQ1
- net N$3 renamed 5VQ2
- net N$5 renamed 5VQ3
Other:
- moved on the sheet: Q1, Q2, Q3, Q4, Q5, Q6, R1, R2, R3, R4, R5, R6
