File: standalone-sensor-board/sensor-board.brd (EAGLE design)
At the start: 26 x 93.5 mm, 32 parts, among them Q1 QRE1113, Q2 QRE1113, Q3 QRE1113, Q4 QRE1113, Q5 QRE1113, Q6 QRE1113, Q7 QRE1113, U1 CD4051BE

Commit message: sensor board
Parts:
- removed D1, D2, D3, D4, D5, D6, D7: 1655, 1655:LED_1655
- removed FFCIN, FFCOUT: 52806-1410, 52806-1410:528061410
- removed RDV: 100k, rcl:0207/10
- removed SJ1, SJ2, SJ3, SJ4, SJ5, SJ6, SJ7: (no value), jumper:SJ
- removed U1: CD4051BE, CD4051BE:N16
- added J1: (no value), 686114148922:686114148922
Connections:
- removed net 3V: D1.3, D2.3, D3.3, D4.3, D5.3, D6.3, D7.3, FFCIN.13, FFCOUT.2
- removed net A: FFCIN.11, FFCOUT.4, U1.11
- removed net B: FFCIN.10, FFCOUT.5, U1.10
- removed net C: FFCIN.9, FFCOUT.6, U1.9
- removed net DIN: D1.2, FFCIN.8
- removed net DOUT: D7.4, FFCOUT.7
- removed net N$15: D6.4, D7.2
- removed net N$16: D1.4, D2.2
- removed net N$17: D2.4, D3.2
- removed net N$18: D3.4, D4.2
- removed net N$19: D4.4, D5.2
- removed net N$2: FFCOUT.3, R1.1, R11.1, R13.1, R3.1, R5.1, R7.1, R9.1
- removed net N$20: D5.4, D6.2
- removed net S1: FFCIN.7, FFCOUT.8, SJ1.1
- removed net S2: FFCIN.6, FFCOUT.9, SJ2.1
- removed net S3: FFCIN.5, FFCOUT.10, SJ3.1
- removed net S4: FFCIN.4, FFCOUT.11, SJ4.1
- removed net S5: FFCIN.3, FFCOUT.12, SJ5.1
- removed net S6: FFCIN.2, FFCOUT.13, SJ6.1
- removed net S7: FFCIN.1, FFCOUT.14, SJ7.1
- removed net SIG: RDV.1, SJ1.2, SJ2.2, SJ3.2, SJ4.2, SJ5.2, SJ6.2, SJ7.2, U1.3
- new net N$4: Q5.1, R9.2
- new net N$6: J1.MP1, J1.MP2
- net C0: now also J1.9; no longer U1.13
- net C1: now also J1.8; no longer U1.14
- net C2: now also J1.7; no longer U1.15
- net C3: now also J1.6; no longer U1.12
- net C4: now also J1.5; no longer U1.1
- net C5: now also J1.4; no longer U1.5
- net C6: now also J1.3; no longer U1.2
- net GND: now also J1.1; no longer D1.1, D2.1, D3.1, D4.1, D5.1, D6.1, D7.1, FFCOUT.1, U1.6, U1.7, U1.8
- net VCC: now also J1.2, R1.1, R11.1, R13.1, R3.1, R5.1, R7.1, R9.1; no longer FFCIN.12, RDV.2, U1.16
Routing:
- net 3V: track 122.7 -> 0.00 mm
- net GND: track 108.9 -> 0.00 mm, vias 7 -> 0
- net S6: track 89.6 -> 0.00 mm, vias 2 -> 0
- net S4: track 88.9 -> 0.00 mm, vias 2 -> 0
- net S2: track 85.8 -> 0.00 mm, vias 2 -> 0
- net S5: track 85.4 -> 0.00 mm, vias 2 -> 0
- net S7: track 80.5 -> 0.00 mm, vias 1 -> 0
- net B: track 79.3 -> 0.00 mm
- net S1: track 79.2 -> 0.00 mm, vias 2 -> 0
- net S3: track 78.6 -> 0.00 mm, vias 2 -> 0
- net C: track 68.1 -> 0.00 mm
- net A: track 65.9 -> 0.00 mm
- net VCC: track 38.2 -> 0.00 mm
- net SIG: track 36.0 -> 0.00 mm
- net DOUT: track 16.7 -> 0.00 mm, vias 1 -> 0
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
Commit message: route
Parts:
- R1, R11, R13, R3, R5, R7, R9: device rcl:0207/10 -> rcl:0204V
- moved J1 61.0 mm to (6.50, 46.8), flipped to the bottom, turned to 270 degrees
- moved R13 56.0 mm to (7.80, 85.7)
- moved R11 44.8 mm to (8.00, 71.8)
- moved R9 35.6 mm to (8.90, 60.5), turned to 270 degrees
- moved R1 14.9 mm to (8.00, 1.70)
- moved R7 10.5 mm to (9.00, 32.7), flipped to the bottom, turned to 90 degrees
- moved R5 8.70 mm to (7.70, 27.6)
- moved R3 5.95 mm to (7.70, 15.5)
Connections:
- removed net N$6: J1.MP1, J1.MP2
- net C0: now also J1.14; no longer J1.9
- net C1: now also J1.13; no longer J1.8
- net C2: now also J1.12; no longer J1.7
- net GND: now also J1.MP1, J1.MP2
Routing:
- net VCC: track 0.00 -> 98.0 mm, vias 0 -> 1
- net N$13: track 60.4 -> 5.69 mm
- net N$11: track 49.1 -> 5.86 mm
- net C1: track 66.8 -> 24.1 mm, vias 3 -> 0
- net C0: track 50.8 -> 36.3 mm
- net N$4: track 0.00 -> 13.5 mm
- net C3: track 11.8 -> 2.35 mm, vias 2 -> 0
- net N$1: track 15.3 -> 5.86 mm
- net N$7: track 25.3 -> 17.4 mm
- net N$5: track 13.6 -> 6.44 mm
- net C6: track 48.3 -> 41.9 mm
- net C2: track 15.8 -> 11.6 mm, vias 2 -> 0
- net N$3: track 7.17 -> 5.65 mm
- net C4: track 18.1 -> 18.6 mm
- net C5: track 29.0 -> 29.1 mm, vias 0 -> 2
Other:
- board size 26 x 93.5 mm -> 11 x 93.5 mm
- board text added: "NEMUS Sensor Board v0.2.0"
- board text removed: "1"
- board text removed: "2"
- board text removed: "3"
- board text removed: "4"
- board text removed: "5"
- board text removed: "6"
- board text removed: "7"
- board text removed: "B"
- board text removed: "NEMUS Face Board v0.1.1"
