File: standalone-sensor-board/sensor-board.sch (EAGLE design)
At the start: 32 parts, among them Q1 QRE1113, Q2 QRE1113, Q3 QRE1113, Q4 QRE1113, Q5 QRE1113, Q6 QRE1113, Q7 QRE1113, U1 CD4051BE

Commit message: sensor board
Parts:
- removed D1, D2, D3, D4, D5, D6, D7: 1655, 1655:1655
- removed FFCIN, FFCOUT: 52806-1410, 52806-1410:52806-1410
- removed RDV: 100k, rcl:R-EU_0207/10
- removed SJ1, SJ2, SJ3, SJ4, SJ5, SJ6, SJ7: (no value), jumper:SJ
- removed U1: CD4051BE, CD4051BE:CD4051BE
- added J1: (no value), 686114148922:686114148922
Connections:
- removed net 3V: D1.VDD, D2.VDD, D3.VDD, D4.VDD, D5.VDD, D6.VDD, D7.VDD, FFCIN.13, FFCOUT.2
- removed net A: FFCIN.11, FFCOUT.4, U1.A
- removed net B: FFCIN.10, FFCOUT.5, U1.B
- removed net C: FFCIN.9, FFCOUT.6, U1.C
- removed net DIN: D1.DIN, FFCIN.8
- removed net DOUT: D7.DOUT, FFCOUT.7
- removed net N$15: D6.DOUT, D7.DIN
- removed net N$16: D1.DOUT, D2.DIN
- removed net N$17: D2.DOUT, D3.DIN
- removed net N$18: D3.DOUT, D4.DIN
- removed net N$19: D4.DOUT, D5.DIN
- removed net N$2: FFCOUT.3, R1.1, R11.1, R13.1, R3.1, R5.1, R7.1, R9.1
- removed net N$20: D5.DOUT, D6.DIN
- removed net S1: FFCIN.7, FFCOUT.8, SJ1.1
- removed net S2: FFCIN.6, FFCOUT.9, SJ2.1
- removed net S3: FFCIN.5, FFCOUT.10, SJ3.1
- removed net S4: FFCIN.4, FFCOUT.11, SJ4.1
- removed net S5: FFCIN.3, FFCOUT.12, SJ5.1
- removed net S6: FFCIN.2, FFCOUT.13, SJ6.1
- removed net S7: FFCIN.1, FFCOUT.14, SJ7.1
- removed net SIG: RDV.1, SJ1.2, SJ2.2, SJ3.2, SJ4.2, SJ5.2, SJ6.2, SJ7.2, U1.COM
- new net N$4: Q5.1, R9.2
- new net N$6: J1.MP1, J1.MP2
- net C0: now also J1.9; no longer U1.CH0
- net C1: now also J1.8; no longer U1.CH1
- net C2: now also J1.7; no longer U1.CH2
- net C3: now also J1.6; no longer U1.CH3
- net C4: now also J1.5; no longer U1.CH4
- net C5: now also J1.4; no longer U1.CH5
- net C6: now also J1.3; no longer U1.CH6
- net GND: now also J1.1; no longer D1.VSS, D2.VSS, D3.VSS, D4.VSS, D5.VSS, D6.VSS, D7.VSS, FFCOUT.1, U1.GND, U1.INH, U1.VEE
- net VCC: now also J1.2, R1.1, R11.1, R13.1, R3.1, R5.1, R7.1, R9.1; no longer FFCIN.12, RDV.2, U1.VDD
Other:
- note removed: "Solder Junction"
- moved on the sheet: R1, R11, R13, R3, R5, R7, R9

Commit message: route
Parts:
- R1, R11, R13, R3, R5, R7, R9: device rcl:R-EU_0207/10 -> rcl:R-EU_0204/2V
Connections:
- removed net N$6: J1.MP1, J1.MP2
- net C0: now also J1.14; no longer J1.9
- net C1: now also J1.13; no longer J1.8
- net C2: now also J1.12; no longer J1.7
- net GND: now also J1.MP1, J1.MP2
Changed lines of the file:
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@@
 <parts>
 <part name="Q1" library="qre1113" deviceset="QRE1113" device=""/>
-<part name="R1" library="rcl" library_urn="urn:adsk.eagle:library:334" deviceset="R-EU_" device="0207/10" package3d_urn="urn:adsk.eagle:package:23491/2" value="100"/>
+<part name="R1" library="rcl" library_urn="urn:adsk.eagle:library:334" deviceset="R-EU_" device="0204/2V" package3d_urn="urn:adsk.eagle:package:23495/1" value="100"/>
 <part name="Q2" library="qre1113" deviceset="QRE1113" device=""/>
-<part name="R3" library="rcl" library_urn="urn:adsk.eagle:library:334" deviceset="R-EU_" device="0207/10" package3d_urn="urn:adsk.eagle:package:23491/2" value="100"/>
+<part name="R3" library="rcl" library_urn="urn:adsk.eagle:library:334" deviceset="R-EU_" device="0204/2V" package3d_urn="urn:adsk.eagle:package:23495/1" value="100"/>
 <part name="Q3" library="qre1113" deviceset="QRE1113" device=""/>
-<part name="R5" library="rcl" library_urn="urn:adsk.eagle:library:334" deviceset="R-EU_" device="0207/10" package3d_urn="urn:adsk.eagle:package:23491/2" value="100"/>
+<part name="R5" library="rcl" library_urn="urn:adsk.eagle:library:334" deviceset="R-EU_" device="0204/2V" package3d_urn="urn:adsk.eagle:package:23495/1" value="100"/>
 <part name="Q4" library="qre1113" deviceset="QRE1113" device=""/>
-<part name="R7" library="rcl" library_urn="urn:adsk.eagle:library:334" deviceset="R-EU_" device="0207/10" package3d_urn="urn:adsk.eagle:package:23491/2" value="100"/>
+<part name="R7" library="rcl" library_urn="urn:adsk.eagle:library:334" deviceset="R-EU_" device="0204/2V" package3d_urn="urn:adsk.eagle:package:23495/1" value="100"/>
 <part name="Q5" library="qre1113" deviceset="QRE1113" device=""/>
-<part name="R9" library="rcl" library_urn="urn:adsk.eagle:library:334" deviceset="R-EU_" device="0207/10" package3d_urn="urn:adsk.eagle:package:23491/2" value="100"/>
+<part name="R9" library="rcl" library_urn="urn:adsk.eagle:library:334" deviceset="R-EU_" device="0204/2V" package3d_urn="urn:adsk.eagle:package:23495/1" value="100"/>
 <part name="Q6" library="qre1113" deviceset="QRE1113" device=""/>
-<part name="R11" library="rcl" library_urn="urn:adsk.eagle:library:334" deviceset="R-EU_" device="0207/10" package3d_urn="urn:adsk.eagle:package:23491/2" value="100"/>
+<part name="R11" library="rcl" library_urn="urn:adsk.eagle:library:334" deviceset="R-EU_" device="0204/2V" package3d_urn="urn:adsk.eagle:package:23495/1" value="100"/>
 <part name="Q7" library="qre1113" deviceset="QRE1113" device=""/>
-<part name="R13" library="rcl" library_urn="urn:adsk.eagle:library:334" deviceset="R-EU_" device="0207/10" package3d_urn="urn:adsk.eagle:package:23491/2" value="100"/>
+<part name="R13" library="rcl" library_urn="urn:adsk.eagle:library:334" deviceset="R-EU_" device="0204/2V" package3d_urn="urn:adsk.eagle:package:23495/1" value="100"/>
 <part name="SUPPLY7" library="supply2" library_urn="urn:adsk.eagle:library:372" deviceset="VCC" device=""/>
 <part name="GND2" library="supply1" library_urn="urn:adsk.eagle:library:371" deviceset="GND" device=""/>
@@
 </instance>
 <instance part="J1" gate="G$1" x="73.66" y="129.54" smashed="yes" rot="R270">
-<attribute name="NAME" x="73.66" y="133.35" size="1.778" layer="95" rot="R270" align="center-left"/>
+<attribute name="NAME" x="81.28" y="107.95" size="1.778" layer="95" rot="R270" align="center-left"/>
 <attribute name="VALUE" x="78.74" y="107.95" size="1.778" layer="96" rot="R270" align="center-left"/>
 </instance>
@@
 </segment>
 <segment>
-<pinref part="J1" gate="G$1" pin="9"/>
-<wire x1="53.34" y1="104.14" x2="53.34" y2="101.6" width="0.1524" layer="91"/>
-<label x="53.34" y="101.6" size="1.778" layer="95" rot="R270" xref="yes"/>
+<label x="40.64" y="101.6" size="1.778" layer="95" rot="R270" xref="yes"/>
+<pinref part="J1" gate="G$1" pin="14"/>
+<wire x1="40.64" y1="101.6" x2="40.64" y2="104.14" width="0.1524" layer="91"/>
 </segment>
 </net>
@@
 <junction x="129.54" y="81.28"/>
 <junction x="134.62" y="81.28"/>
-<pinref part="J1" gate="G$1" pin="1"/>
 <wire x1="134.62" y1="88.9" x2="134.62" y2="81.28" width="0.1524" layer="91"/>
 <wire x1="73.66" y1="104.14" x2="73.66" y2="88.9" width="0.1524" layer="91"/>
-<wire x1="73.66" y1="88.9" x2="134.62" y2="88.9" width="0.1524" layer="91"/>
+<wire x1="73.66" y1="88.9" x2="78.74" y2="88.9" width="0.1524" layer="91"/>
+<wire x1="78.74" y1="88.9" x2="134.62" y2="88.9" width="0.1524" layer="91"/>
+<wire x1="71.12" y1="129.54" x2="73.66" y2="129.54" width="0.1524" layer="91"/>
+<wire x1="73.66" y1="129.54" x2="78.74" y2="129.54" width="0.1524" layer="91"/>
+<wire x1="78.74" y1="129.54" x2="78.74" y2="88.9" width="0.1524" layer="91"/>
+<junction x="78.74" y="88.9"/>
+<pinref part="J1" gate="G$1" pin="1"/>
+<pinref part="J1" gate="G$1" pin="MP1"/>
+<junction x="73.66" y="129.54"/>
+<pinref part="J1" gate="G$1" pin="MP2"/>
 </segment>
 </net>
@@
 </segment>
 <segment>
-<pinref part="J1" gate="G$1" pin="8"/>
-<wire x1="55.88" y1="104.14" x2="55.88" y2="96.52" width="0.1524" layer="91"/>
-<label x="55.88" y="96.52" size="1.778" layer="95" rot="R270" xref="yes"/>
+<label x="43.18" y="96.52" size="1.778" layer="95" rot="R270" xref="yes"/>
+<pinref part="J1" gate="G$1" pin="13"/>
+<wire x1="43.18" y1="96.52" x2="43.18" y2="104.14" width="0.1524" layer="91"/>
 </segment>
 </net>
@@
 </segment>
 <segment>
-<pinref part="J1" gate="G$1" pin="7"/>
-<wire x1="58.42" y1="104.14" x2="58.42" y2="101.6" width="0.1524" layer="91"/>
-<label x="58.42" y="101.6" size="1.778" layer="95" rot="R270" xref="yes"/>
+<label x="45.72" y="101.6" size="1.778" layer="95" rot="R270" xref="yes"/>
+<pinref part="J1" gate="G$1" pin="12"/>
+<wire x1="45.72" y1="101.6" x2="45.72" y2="104.14" width="0.1524" layer="91"/>
 </segment>
 </net>
@@
 </segment>
 <segment>
-<pinref part="J1" gate="G$1" pin="6"/>
 <wire x1="60.96" y1="104.14" x2="60.96" y2="96.52" width="0.1524" layer="91"/>
 <label x="60.96" y="96.52" size="1.778" layer="95" rot="R270" xref="yes"/>
+<pinref part="J1" gate="G$1" pin="6"/>
 </segment>
 </net>
@@
 </segment>
 <segment>
-<pinref part="J1" gate="G$1" pin="5"/>
 <wire x1="63.5" y1="104.14" x2="63.5" y2="101.6" width="0.1524" layer="91"/>
 <label x="63.5" y="101.6" size="1.778" layer="95" rot="R270" xref="yes"/>
+<pinref part="J1" gate="G$1" pin="5"/>
 </segment>
 </net>
@@
 </segment>
 <segment>
-<pinref part="J1" gate="G$1" pin="4"/>
 <wire x1="66.04" y1="104.14" x2="66.04" y2="96.52" width="0.1524" layer="91"/>
 <label x="66.04" y="96.52" size="1.778" layer="95" rot="R270" xref="yes"/>
+<pinref part="J1" gate="G$1" pin="4"/>
 </segment>
 </net>
@@
 </segment>
 <segment>
-<pinref part="J1" gate="G$1" pin="3"/>
 <wire x1="68.58" y1="104.14" x2="68.58" y2="101.6" width="0.1524" layer="91"/>
 <label x="68.58" y="101.6" size="1.778" layer="95" rot="R270" xref="yes"/>
+<pinref part="J1" gate="G$1" pin="3"/>
 </segment>
 </net>
@@
 <pinref part="R9" gate="G$1" pin="2"/>
 <wire x1="73.66" y1="71.12" x2="73.66" y2="73.66" width="0.1524" layer="91"/>
-</segment>
-</net>
-<net name="N$6" class="0">
-<segment>
-<pinref part="J1" gate="G$1" pin="MP2"/>
-<pinref part="J1" gate="G$1" pin="MP1"/>
-<wire x1="71.12" y1="129.54" x2="73.66" y2="129.54" width="0.1524" layer="91"/>
 </segment>
 </net>
@@
 <wire x1="139.7" y1="60.96" x2="114.3" y2="60.96" width="0.1524" layer="91"/>
 <junction x="114.3" y="60.96"/>
-<pinref part="J1" gate="G$1" pin="2"/>
 <wire x1="71.12" y1="104.14" x2="71.12" y2="83.82" width="0.1524" layer="91"/>
 <wire x1="71.12" y1="83.82" x2="-15.24" y2="83.82" width="0.1524" layer="91"/>
@@
 <wire x1="-15.24" y1="60.96" x2="-10.16" y2="60.96" width="0.1524" layer="91"/>
 <junction x="-10.16" y="60.96"/>
+<pinref part="J1" gate="G$1" pin="2"/>
 </segment>
 </net>
@@
 </sheet>
 </sheets>
+<errors>
+</errors>
 </schematic>
 </drawing>

Commit message: tidy silk screen
Parts:
- R1, R11, R13, R3, R5, R7, R9: device rcl:R-EU_0204/2V -> rcl:R-EU_0207/10
Changed lines of the file:
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@@
 <parts>
 <part name="Q1" library="qre1113" deviceset="QRE1113" device=""/>
-<part name="R1" library="rcl" library_urn="urn:adsk.eagle:library:334" deviceset="R-EU_" device="0204/2V" package3d_urn="urn:adsk.eagle:package:23495/1" value="100"/>
+<part name="R1" library="rcl" library_urn="urn:adsk.eagle:library:334" deviceset="R-EU_" device="0207/10" package3d_urn="urn:adsk.eagle:package:23491/2" value="100"/>
 <part name="Q2" library="qre1113" deviceset="QRE1113" device=""/>
-<part name="R3" library="rcl" library_urn="urn:adsk.eagle:library:334" deviceset="R-EU_" device="0204/2V" package3d_urn="urn:adsk.eagle:package:23495/1" value="100"/>
+<part name="R3" library="rcl" library_urn="urn:adsk.eagle:library:334" deviceset="R-EU_" device="0207/10" package3d_urn="urn:adsk.eagle:package:23491/2" value="100"/>
 <part name="Q3" library="qre1113" deviceset="QRE1113" device=""/>
-<part name="R5" library="rcl" library_urn="urn:adsk.eagle:library:334" deviceset="R-EU_" device="0204/2V" package3d_urn="urn:adsk.eagle:package:23495/1" value="100"/>
+<part name="R5" library="rcl" library_urn="urn:adsk.eagle:library:334" deviceset="R-EU_" device="0207/10" package3d_urn="urn:adsk.eagle:package:23491/2" value="100"/>
 <part name="Q4" library="qre1113" deviceset="QRE1113" device=""/>
-<part name="R7" library="rcl" library_urn="urn:adsk.eagle:library:334" deviceset="R-EU_" device="0204/2V" package3d_urn="urn:adsk.eagle:package:23495/1" value="100"/>
+<part name="R7" library="rcl" library_urn="urn:adsk.eagle:library:334" deviceset="R-EU_" device="0207/10" package3d_urn="urn:adsk.eagle:package:23491/2" value="100"/>
 <part name="Q5" library="qre1113" deviceset="QRE1113" device=""/>
-<part name="R9" library="rcl" library_urn="urn:adsk.eagle:library:334" deviceset="R-EU_" device="0204/2V" package3d_urn="urn:adsk.eagle:package:23495/1" value="100"/>
+<part name="R9" library="rcl" library_urn="urn:adsk.eagle:library:334" deviceset="R-EU_" device="0207/10" package3d_urn="urn:adsk.eagle:package:23491/2" value="100"/>
 <part name="Q6" library="qre1113" deviceset="QRE1113" device=""/>
-<part name="R11" library="rcl" library_urn="urn:adsk.eagle:library:334" deviceset="R-EU_" device="0204/2V" package3d_urn="urn:adsk.eagle:package:23495/1" value="100"/>
+<part name="R11" library="rcl" library_urn="urn:adsk.eagle:library:334" deviceset="R-EU_" device="0207/10" package3d_urn="urn:adsk.eagle:package:23491/2" value="100"/>
 <part name="Q7" library="qre1113" deviceset="QRE1113" device=""/>
-<part name="R13" library="rcl" library_urn="urn:adsk.eagle:library:334" deviceset="R-EU_" device="0204/2V" package3d_urn="urn:adsk.eagle:package:23495/1" value="100"/>
+<part name="R13" library="rcl" library_urn="urn:adsk.eagle:library:334" deviceset="R-EU_" device="0207/10" package3d_urn="urn:adsk.eagle:package:23491/2" value="100"/>
 <part name="SUPPLY7" library="supply2" library_urn="urn:adsk.eagle:library:372" deviceset="VCC" device=""/>
 <part name="GND2" library="supply1" library_urn="urn:adsk.eagle:library:371" deviceset="GND" device=""/>
